Commit message: set joint limits + define gazebo plugin

File: urdf/example_manipulator.urdf.xacro (robot description, xacro)
@@ -18,5 +18,5 @@
         </link>
     </xacro:macro>
-    <xacro:macro name="make_cont_joint" params="name parent child xyz rpy">
+    <xacro:macro name="make_cont_joint" params="name parent child xyz rpy effort velocity">
         <joint name="${name}" type="continuous">
             <parent link="${parent}" />
@@ -24,4 +24,5 @@
             <origin xyz="${xyz}" rpy="${rpy}" />
             <axis xyz="0 0 1" />
+            <limit effort="${effort}" velocity="${velocity}" />
         </joint>
         <transmission name="${name}_trans">
@@ -39,9 +40,21 @@
     <!-- Links & joints -->
     <xacro:make_box_link name="body" mass="1." size_x="0.2" size_y="0.2" size_z="0.2" />
-    <xacro:make_cont_joint name="shoulder" parent="body" child="upper_arm" xyz="0.2 0 0" rpy="${90 * TORAD} 0 0" />
+    <xacro:make_cont_joint name="shoulder" parent="body" child="upper_arm"
+                           xyz="0.2 0 0" rpy="${90 * TORAD} 0 0"
+                           effort="30." velocity="1." />
     <xacro:make_box_link name="upper_arm" mass="1." size_x="0.3" size_y="0.1" size_z="0.1" />
-    <xacro:make_cont_joint name="elbow" parent="upper_arm" child="forearm" xyz="0.3 0 0" rpy="0 0 0" />
+    <xacro:make_cont_joint name="elbow" parent="upper_arm" child="forearm"
+                           xyz="0.3 0 0" rpy="0 0 0"
+                           effort="15." velocity="1." />
     <xacro:make_box_link name="forearm" mass="1." size_x="0.3" size_y="0.05" size_z="0.05" />
-    <xacro:make_cont_joint name="wrist" parent="forearm" child="hand" xyz="0.3 0 0" rpy="0 0 0" />
+    <xacro:make_cont_joint name="wrist" parent="forearm" child="hand"
+                           xyz="0.3 0 0" rpy="0 0 0"
+                           effort="5." velocity="1." />
     <xacro:make_box_link name="hand" mass="0.3" size_x="0.1" size_y="0.1" size_z="0.1" />
+    <!-- Gazebo plugin -->
+    <gazebo>
+        <plugin name="gazebo_ros_control" filename="libgazebo_ros_control.so">
+            <legacyModeNS>false</legacyModeNS>
+        </plugin>
+    </gazebo>
 </robot>

Commit message: match model root joint in gazebo & urdf (fix base link to world)

File: urdf/example_manipulator.urdf.xacro (robot description, xacro)
@@ -1,3 +1,6 @@
 <robot name="example_manipulator" xmlns:xacro="http://wiki.ros.org/xacro">
+    <!-- Args -->
+    <xacro:arg name="fixed_base_link" default="false" />
+    <xacro:property name="do_fix_base_link" value="$(arg fixed_base_link)" />
     <!-- Macros -->
     <xacro:macro name="make_box_link" params="name mass size_x size_y size_z">
@@ -39,4 +42,19 @@
     <xacro:property name="TORAD" value="${3.14159265359 / 180}" />
     <!-- Links & joints -->
+    <xacro:if value="${do_fix_base_link}">
+        <link name="world">
+            <inertial>
+                <origin xyz="0 0 0" />
+                <mass value="1000" />
+                <inertia ixx="100" ixy="0" ixz="0"
+                         iyy="100" iyz="0"
+                         izz="100" />
+            </inertial>
+        </link>
+        <joint name="anchor" type="fixed">
+            <parent link="world" />
+            <child link="body" />
+        </joint>
+    </xacro:if>
     <xacro:make_box_link name="body" mass="1." size_x="0.2" size_y="0.2" size_z="0.2" />
     <xacro:make_cont_joint name="shoulder" parent="body" child="upper_arm"
